File: Mainboard/KiCad/Omega-Mainboard.kicad_pcb (KiCad board)
At the start: 2 copper layers, 333.4 x 149.9 mm, 238 parts, among them J1 5V, J10 POWER, J11 KEYBOARD, J12 RAM_EXT, J2 Composite, J3 Audio, J4 S-VIDEO, J5 RGB, J6 Cassette, J7 JOYSTICK_A, J8 JOYSTICK_B, J9 PRINTER, Q1 PN2907A, Q2 PN2222A, U1 Z84C00, U10 D41464, U11 D41464, U12 ATF16V8B, U13 ATF16V8B, U14 ATF16V8B, U15 74HCT670, U16 74HCT670, U17 74HCT670, U18 74HCT670, U19 74F541, U2 82C55, U20 74F541, U21 74F541, U22 74HCT540, U23 74HCT273, U24 74HCT273, U25 74F245, U26 74F245, U27 74HCT175, U28 74HCT157, U29 74HCT157, U3 V9938, U30 74HCT153, U31 74HCT153, U32 74AHCT138, U33 74AHCT125, U34 74HCT74, U35 74HCT74, U36 74HCT74, U37 74AHCT32, U38 74AHCT32, U39 74AHCT32, U4 YM2149, U40 74HCT30, U41 74HCT30, U42 74LS07, U43 74HCT04, U44 74AHCT02, U45 74HCT00, U46 ADM693, U47 CXA1645, U48 OPA340P, U49 LM311, U5 RP5C01, U6 SST39SF040, U7 AS6C4008, U8 D41464, U9 D41464, Y1 21.477270MHz, Y2 32768 Hz, Y3 4.433618MHz

Commit message: Mainboard: Fix the issues discovered so far
Signed-off-by: Sergey Kiselev <skiselev@gmail.com>
Connections:
- U37 pad 1: /Memory/~PAGE_WR -> /~RD
- U37 pad 10: /Processor/~PRT_STB_WR -> /Processor/~PRT_CMD_CS
- U37 pad 11: /~RD -> /Memory/~PAGE_WR
- U37 pad 13: /Memory/~PAGE_RD -> /~WR
- U37 pad 3: /~WR -> /Memory/~PAGE_RD
- U37 pad 4: /Processor/~PRT_BSY_RD -> /~RD
- U37 pad 5: /~RD -> /Processor/~PRT_CMD_CS
- U37 pad 6: /Processor/~PRT_CMD_CS -> /Processor/~PRT_BSY_RD
- U37 pad 8: /~WR -> /Processor/~PRT_STB_WR
- U37 pad 9: /Processor/~PRT_CMD_CS -> /~WR
- U38 pad 1: /PPI/~SUB_REG_CS -> /PPI/~SLTSL3
- U38 pad 10: /PPI/~SUB_RD -> /PPI/~SUB_REG_CS
- U38 pad 11: /PPI/~SUB_REG_CS -> /PPI/~SUB_RD
- U38 pad 12: /~RD -> /PPI/~SUB_REG_CS
- U38 pad 13: /PPI/~SUB_WR -> /~RD
- U38 pad 2: /PPI/~SLTSL3 -> /PPI/~FFFF
- U38 pad 3: /PPI/~FFFF -> /PPI/~SUB_REG_CS
- U38 pad 4: /PPI/~FFFF -> Net-(U38-Pad4)
- U38 pad 6: Net-(U38-Pad6) -> /PPI/~FFFF
- U38 pad 8: /~WR -> /PPI/~SUB_WR
- U38 pad 9: /PPI/~SUB_REG_CS -> /~WR
- U39 pad 1: /CLK -> /~RD
- U39 pad 10: /VDP/~VDP_WR -> Net-(U39-Pad10)
- U39 pad 11: Net-(U39-Pad11) -> /VDP/~VDP_WR
- U39 pad 12: /~PSG_CS -> /~WR
- U39 pad 13: Net-(U39-Pad13) -> /~VDP_CS
- U39 pad 2: /CLK -> /~VDP_CS
- U39 pad 3: Net-(JP5-Pad1) -> /VDP/~VDP_RD
- U39 pad 4: /VDP/~VDP_RD -> /CLK
- U39 pad 5: /~RD -> /CLK
- U39 pad 6: /~VDP_CS -> Net-(JP5-Pad1)
- U39 pad 8: /~WR -> Net-(U39-Pad8)
- U39 pad 9: /~VDP_CS -> /~PSG_CS
- U40 pad 8: Net-(U38-Pad6) -> Net-(U38-Pad5)
- U41 pad 8: Net-(U38-Pad5) -> Net-(U38-Pad4)
- U44 pad 1: Net-(U36-Pad1) -> Net-(U39-Pad10)
- U44 pad 12: Net-(U39-Pad13) -> Net-(U39-Pad8)
- U44 pad 2: /~PSG_CS -> Net-(U36-Pad8)
- U44 pad 3: /~PSG_CS -> Net-(RR6-Pad10)
- U44 pad 4: Net-(U39-Pad11) -> Net-(U36-Pad1)
- U44 pad 5: Net-(U36-Pad8) -> /~PSG_CS
- U44 pad 6: Net-(RR6-Pad10) -> /~PSG_CS
- U44 pad 8: Net-(U39-Pad13) -> Net-(U39-Pad8)
Routing:
- net Net-(U38-Pad4): track 0.00 -> 188.1 mm, vias 0 -> 1
- net Net-(U38-Pad5): track 185.6 -> 35.1 mm, vias 1 -> 0
- net Net-(U38-Pad6): track 43.4 -> 0.00 mm
- net GND: track 4233.3 -> 4261.7 mm
- net Net-(U39-Pad8): track 0.00 -> 25.0 mm
- net Net-(U39-Pad13): track 25.0 -> 0.00 mm
- net Net-(U39-Pad10): track 0.00 -> 15.9 mm, vias 0 -> 1
- net /PPI/~SUB_WR: track 164.7 -> 179.0 mm
- net VCC: track 2267.9 -> 2280.8 mm
- net Net-(U36-Pad1): track 44.1 -> 31.5 mm
- net /Memory/~PAGE_WR: track 249.4 -> 259.3 mm
- net /~WR: track 356.4 -> 346.6 mm, vias 6 -> 5
- net /~VDP_CS: track 38.8 -> 29.4 mm
- net /~PSG_CS: track 39.8 -> 48.0 mm
- net /PPI/~FFFF: track 31.1 -> 38.7 mm
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Other:
- board text added: "Omega Home Computer Main Board - Version 1.1 Copyright (C) 2018-2019 Sergey Kiselev"
- board text added: "github.com/skiselev/omega www.malinov.com"
- board text removed: "Omega Home Computer Main Board - Version 1.0 Copyright (C) 2018-2019 Sergey Kiselev"

Commit message: Mainboard: Fixed schematic and PCB for v1.1
Signed-off-by: Sergey Kiselev <skiselev@gmail.com>
Parts:
- removed the C83 at (106.7, 47.0)
- removed the R31 at (45.7, 54.6)
- added C59: 0.1uF, My_Components:Cap_Cer_508, F.Cu at (134.6, 58.4)
- added R20: 4.7k, My_Components:Res_762, F.Cu at (123.2, 55.9)
- added R21: 4.7k, My_Components:Res_762, F.Cu at (123.2, 58.4)
- added R22: 4.7k, My_Components:Res_762, F.Cu at (198.1, 45.7)
- added R23: 4.7k, My_Components:Res_762, F.Cu at (200.7, 45.7)
- added R24: 4.7k, My_Components:Res_762, F.Cu at (203.2, 45.7)
- added R48: 0, My_Components:Res_762, F.Cu at (63.5, 21.6)
- C91: value 30pF -> 27pF
- J9: footprint My_Components:Conn_Dsub_DB25F -> My_Components:Conn_Micro_Ribbon_14F
- Q2: value PN2222A -> PN2907A
- R29: renamed from R22; value 2.2k -> 1k
- R30: value 270 -> 1k
- moved C15 71.1 mm to (241.3, 102.9)
- moved C16 71.1 mm to (241.3, 138.4)
- moved C17 71.1 mm to (241.3, 123.2)
- moved C18 71.1 mm to (241.3, 153.7)
- moved C25 71.1 mm to (241.3, 72.4)
- moved C26 71.1 mm to (241.3, 87.6)
- moved RR4 71.1 mm to (257.8, 63.5)
- moved U25 71.1 mm to (257.8, 72.4)
- moved U26 71.1 mm to (257.8, 87.6)
- moved U15 71.1 mm to (255.3, 102.9)
- moved U16 71.1 mm to (255.3, 138.4)
- moved U17 71.1 mm to (255.3, 123.2)
- moved U18 71.1 mm to (255.3, 153.7)
- moved U20 66.0 mm to (323.9, 67.3)
- moved C20 66.0 mm to (307.3, 67.3)
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- renumbered C59 to C60, C60 to C61, C61 to C62, C62 to C63, C63 to C64, C64 to C65, C65 to C66, C66 to C67, C67 to C68, C68 to C69, C69 to C70, C70 to C71, C71 to C72, C72 to C73, C73 to C74, C74 to C75, C75 to C76, C76 to C77, C77 to C78, C78 to C79, C79 to C80, C80 to C81, C81 to C82, C82 to C83, R20 to R25, R21 to R26, R23 to R27, R24 to R28, R25 to R31, R26 to R32, R27 to R33, R28 to R34, R29 to R35, R32 to R36, R33 to R37, R34 to R38, R35 to R39, R36 to R40, R37 to R41, R38 to R42, R39 to R43, R40 to R44, R41 to R45, R42 to R46, R43 to R47
Connections:
- C88 pad 1: Net-(C88-Pad1) -> /VDP/SYNCIN
- J12 pad 10: /A13 -> /Memory/~RAM7_CS
- J12 pad 11: /A7 -> /Memory/RAM_A16
- J12 pad 12: /A8 -> /Memory/RAM_A15
- J12 pad 13: /A6 -> /Memory/RAM_A14
- J12 pad 14: /A9 -> /Memory/RAM_A17
- J12 pad 15: /A5 -> /A12
- J12 pad 16: /A11 -> /~WR
- J12 pad 17: /A4 -> /A7
- J12 pad 18: /~RD -> /A13
- J12 pad 19: /A3 -> /A6
- J12 pad 20: /A10 -> /A8
- J12 pad 21: /A2 -> /A5
- J12 pad 22: /Memory/MD7 -> /A9
- J12 pad 23: /A1 -> /A4
- J12 pad 24: /Memory/MD6 -> /A11
- J12 pad 25: /A0 -> /A3
- J12 pad 26: /Memory/MD5 -> /~RD
- J12 pad 27: /Memory/MD0 -> /A2
- J12 pad 28: /Memory/MD4 -> /A10
- J12 pad 29: /Memory/MD1 -> /A1
- J12 pad 3: /Memory/RAM_A18 -> /Memory/~RAM2_CS
- J12 pad 30: /Memory/MD3 -> /Memory/MD7
- J12 pad 31: /Memory/MD2 -> /A0
- J12 pad 32: /Memory/~RAM1_CS -> /Memory/MD6
- J12 pad 33: /Memory/~RAM2_CS -> /Memory/MD0
- J12 pad 34: /Memory/~RAM3_CS -> /Memory/MD5
- J12 pad 35: /Memory/~RAM4_CS -> /Memory/MD1
- J12 pad 36: /Memory/~RAM5_CS -> /Memory/MD4
- J12 pad 37: /Memory/~RAM6_CS -> /Memory/MD2
- J12 pad 38: /Memory/~RAM7_CS -> /Memory/MD3
- J12 pad 4: /Memory/RAM_A15 -> /Memory/~RAM1_CS
- J12 pad 5: /Memory/RAM_A16 -> /Memory/~RAM4_CS
- J12 pad 6: /Memory/RAM_A17 -> /Memory/~RAM3_CS
- J12 pad 7: /Memory/RAM_A14 -> /Memory/~RAM6_CS
- J12 pad 8: /~WR -> /Memory/~RAM5_CS
- J12 pad 9: /A12 -> /Memory/RAM_A18
- J5 pad 8: /VDP/SYNC -> Net-(J5-Pad8)
- J9 pad 14: Net-(J9-Pad14) -> GND
- Q2 pad 1: Net-(Q2-Pad1) -> VCC
- Q2 pad 2: /VDP/CSYNC -> Net-(Q2-Pad2)
- Q2 pad 3: VCC -> Net-(Q2-Pad3)
- R29 pad 1: Net-(C88-Pad1) -> Net-(Q2-Pad2)
- R30 pad 2: Net-(Q2-Pad1) -> Net-(Q2-Pad3)
- RR2 pad 7: Net-(RR2-Pad7) -> /~VDP_INT
- RR4 pad 10: Net-(RR4-Pad10) -> /Slots/BD0
- RR4 pad 2: /Slots/BD0 -> Net-(RR4-Pad2)
- RR4 pad 3: /Slots/BD1 -> /Slots/BD7
- RR4 pad 4: /Slots/BD2 -> /Slots/BD6
- RR4 pad 5: /Slots/BD3 -> /Slots/BD5
- RR4 pad 7: /Slots/BD5 -> /Slots/BD3
- RR4 pad 8: /Slots/BD6 -> /Slots/BD2
- RR4 pad 9: /Slots/BD7 -> /Slots/BD1
- RR5 pad 10: /~BUSDIR2 -> /~SLT_WAIT
- RR5 pad 2: /Processor/~BUSREQ -> /~KBD_WAIT
- RR5 pad 3: /Processor/~NMI -> /Processor/PRT_BUSY
- RR5 pad 4: /~VDP_WAIT -> /Processor/~BUSREQ
- RR5 pad 5: /~KBD_WAIT -> /Processor/~NMI
- RR5 pad 6: /Processor/PRT_BUSY -> /~BUSDIR1
- RR5 pad 7: /~BUSDIR1 -> /~BUSDIR2
- RR5 pad 8: /~SLT_INT -> Net-(RR5-Pad8)
- RR5 pad 9: /~SLT_WAIT -> /~SLT_INT
- SLOT1 pad 44: Net-(SLOT1-Pad44) -> GND
- SLOT1 pad 46: Net-(SLOT1-Pad44) -> Net-(SLOT1-Pad46)
- SLOT2 pad 44: Net-(SLOT2-Pad44) -> GND
- SLOT2 pad 46: Net-(SLOT2-Pad44) -> Net-(SLOT2-Pad46)
- U14 pad 13: /Slots/~CS1 -> /Slots/~CS12
- U14 pad 14: /Slots/~CS2 -> /Slots/~CS1
- U14 pad 15: /Slots/~CS12 -> /Slots/~CS2
- U15 pad 1: /D0 -> /D7
- U15 pad 10: /D1 -> /D6
- U15 pad 15: /D1 -> /D6
- U15 pad 2: /D2 -> /D5
- U15 pad 3: /D3 -> /D4
- U15 pad 6: /D3 -> /D4
- U15 pad 7: /D2 -> /D5
- U15 pad 9: /D0 -> /D7
- U16 pad 1: /D4 -> /D2
- U16 pad 10: /D5 -> /D3
- U16 pad 15: /D5 -> /D3
- U16 pad 2: /D6 -> /D1
- U16 pad 3: /D7 -> /D0
- U16 pad 6: /D7 -> /D0
- U16 pad 7: /D6 -> /D1
- U16 pad 9: /D4 -> /D2
- U17 pad 1: /D0 -> /D7
- U17 pad 10: /Memory/RAM_A15 -> /Memory/RAM_A20
- U17 pad 15: /D1 -> /D6
- U17 pad 2: /D2 -> /D5
- U17 pad 3: /D3 -> /D4
- U17 pad 6: /Memory/RAM_A17 -> /Memory/RAM_A18
- U17 pad 7: /Memory/RAM_A16 -> /Memory/RAM_A19
- U17 pad 9: /Memory/RAM_A14 -> /Memory/RAM_A21
- U18 pad 1: /D4 -> /D2
- U18 pad 10: /Memory/RAM_A19 -> /Memory/RAM_A17
- U18 pad 15: /D5 -> /D3
- U18 pad 2: /D6 -> /D1
- U18 pad 3: /D7 -> /D0
- U18 pad 6: /Memory/RAM_A21 -> /Memory/RAM_A14
- U18 pad 7: /Memory/RAM_A20 -> /Memory/RAM_A15
- U18 pad 9: /Memory/RAM_A18 -> /Memory/RAM_A16
- U19 pad 11: /Slots/BA5 -> /Slots/BA13
- U19 pad 12: /Slots/BA4 -> /Slots/BA14
- U19 pad 13: /Slots/BA3 -> /Slots/BA0
- U19 pad 14: /Slots/BA2 -> /Slots/BA1
- U19 pad 15: /Slots/BA1 -> /Slots/BA2
- U19 pad 16: /Slots/BA0 -> /Slots/BA3
- U19 pad 17: /Slots/BA14 -> /Slots/BA4
- U19 pad 18: /Slots/BA13 -> /Slots/BA5
- U19 pad 2: /A13 -> /A5
- U19 pad 3: /A14 -> /A4
- U19 pad 4: /A0 -> /A3
- U19 pad 5: /A1 -> /A2
- U19 pad 6: /A2 -> /A1
- U19 pad 7: /A3 -> /A0
- U19 pad 8: /A4 -> /A14
- U19 pad 9: /A5 -> /A13
- U20 pad 11: /Slots/BA12 -> /Slots/BA15
- U20 pad 12: /Slots/BA8 -> /Slots/BA9
- U20 pad 13: /Slots/BA7 -> /Slots/BA10
- U20 pad 14: /Slots/BA6 -> /Slots/BA11
- U20 pad 15: /Slots/BA11 -> /Slots/BA6
- U20 pad 16: /Slots/BA10 -> /Slots/BA7
- U20 pad 17: /Slots/BA9 -> /Slots/BA8
- U20 pad 18: /Slots/BA15 -> /Slots/BA12
- U20 pad 2: /A15 -> /A12
- U20 pad 3: /A9 -> /A8
- U20 pad 4: /A10 -> /A7
- U20 pad 5: /A11 -> /A6
- U20 pad 6: /A6 -> /A11
- U20 pad 7: /A7 -> /A10
- U20 pad 8: /A8 -> /A9
- U20 pad 9: /A12 -> /A15
- U21 pad 11: /Slots/~B_RESET -> /Slots/B_CLK
- U21 pad 12: /Slots/~B_WR -> /Slots/~B_RESET
- U21 pad 13: /Slots/~B_RD -> /Slots/~B_RFSH
- U21 pad 14: /Slots/~B_IORQ -> /Slots/~B_MREQ
- U21 pad 15: /Slots/~B_MREQ -> /Slots/~B_IORQ
- U21 pad 17: /Slots/~B_RFSH -> /Slots/~B_WR
- U21 pad 18: /Slots/B_CLK -> /Slots/~B_RD
- U21 pad 2: /CLK -> /~RD
- U21 pad 3: /~RFSH -> /~WR
- U21 pad 5: /~MREQ -> /~IORQ
- U21 pad 6: /~IORQ -> /~MREQ
- U21 pad 7: /~RD -> /~RFSH
- U21 pad 8: /~WR -> /~RESET
- U21 pad 9: /~RESET -> /CLK
- U24 pad 12: /Processor/PD6 -> /Processor/PD4
- U24 pad 13: /D6 -> /D4
- U24 pad 14: /D4 -> /D1
- U24 pad 15: /Processor/PD4 -> /Processor/PD1
- U24 pad 16: /Processor/PD2 -> /Processor/PD0
- U24 pad 17: /D2 -> /D0
- U24 pad 18: /D0 -> /D6
- U24 pad 19: /Processor/PD0 -> /Processor/PD6
- U24 pad 2: /Processor/PD1 -> /Processor/PD7
- U24 pad 3: /D1 -> /D7
- U24 pad 4: /D3 -> /D2
- U24 pad 5: /Processor/PD3 -> /Processor/PD2
- U24 pad 6: /Processor/PD5 -> /Processor/PD3
- U24 pad 7: /D5 -> /D3
- U24 pad 8: /D7 -> /D5
- U24 pad 9: /Processor/PD7 -> /Processor/PD5
- U25 pad 11: /Slots/BD7 -> /Slots/BD0
- U25 pad 12: /Slots/BD6 -> /Slots/BD1
- U25 pad 13: /Slots/BD5 -> /Slots/BD2
- U25 pad 14: /Slots/BD4 -> /Slots/BD3
- U25 pad 15: /Slots/BD3 -> /Slots/BD4
- U25 pad 16: /Slots/BD2 -> /Slots/BD5
- U25 pad 17: /Slots/BD1 -> /Slots/BD6
- U25 pad 18: /Slots/BD0 -> /Slots/BD7
- U25 pad 2: /D0 -> /D7
- U25 pad 3: /D1 -> /D6
- U25 pad 4: /D2 -> /D5
- U25 pad 5: /D3 -> /D4
- U25 pad 6: /D4 -> /D3
- U25 pad 7: /D5 -> /D2
- U25 pad 8: /D6 -> /D1
- U25 pad 9: /D7 -> /D0
- U26 pad 11: /Memory/MD7 -> /Memory/MD0
- U26 pad 12: /Memory/MD6 -> /Memory/MD1
- U26 pad 13: /Memory/MD5 -> /Memory/MD2
- U26 pad 14: /Memory/MD4 -> /Memory/MD3
- U26 pad 15: /Memory/MD3 -> /Memory/MD4
- U26 pad 16: /Memory/MD2 -> /Memory/MD5
- U26 pad 17: /Memory/MD1 -> /Memory/MD6
- U26 pad 18: /Memory/MD0 -> /Memory/MD7
- U26 pad 2: /D0 -> /D7
- U26 pad 3: /D1 -> /D6
- U26 pad 4: /D2 -> /D5
- U26 pad 5: /D3 -> /D4
- U26 pad 6: /D4 -> /D3
- U26 pad 7: /D5 -> /D2
- U26 pad 8: /D6 -> /D1
- U26 pad 9: /D7 -> /D0
- U27 pad 4: /D0 -> /D1
- U27 pad 5: /D1 -> /D0
- U35 pad 10: /~RESET -> VCC
- U35 pad 11: /Processor/~PRT_STB_WR -> /CLK
- U35 pad 12: /D0 -> Net-(U35-Pad12)
- U35 pad 2: /CLK -> /D0
- U35 pad 3: Net-(U35-Pad3) -> /Processor/~PRT_STB_WR
- U35 pad 4: VCC -> /~RESET
- U35 pad 5: Net-(U35-Pad5) -> /Processor/~STROBE
- U35 pad 6: Net-(U35-Pad3) -> Net-(U35-Pad6)
- U35 pad 8: Net-(U35-Pad8) -> Net-(U35-Pad12)
- U35 pad 9: /Processor/~STROBE -> Net-(U35-Pad9)
- U4 pad 22: Net-(U35-Pad5) -> Net-(U35-Pad9)
- U41 pad 11: /A13 -> /A8
- U41 pad 12: /A12 -> /A13
- U41 pad 3: /A8 -> /A12
- U41 pad 4: /A9 -> /A10
- U41 pad 5: /A11 -> /A9
- U41 pad 6: /A10 -> /A11
- U43 pad 5: GND -> Net-(Q2-Pad3)
- U43 pad 6: Net-(U43-Pad6) -> /VDP/SYNCIN
- U47 pad 10: Net-(C88-Pad1) -> /VDP/SYNCIN
- U48 pad 3: GND -> Net-(C59-Pad1)
- U5 pad 4: Net-(U27-Pad2) -> Net-(U27-Pad7)
- U5 pad 5: Net-(U27-Pad7) -> Net-(U27-Pad2)
Routing:
- net GND: track 4261.7 -> 4713.7 mm, vias 29 -> 41
- net /D6: track 490.1 -> 353.7 mm, vias 0 -> 1
- net /~VDP_WAIT: track 252.8 -> 129.2 mm, vias 3 -> 1
- net /D7: track 447.1 -> 323.7 mm
- net /D4: track 487.6 -> 371.7 mm, vias 2 -> 1
- net /D5: track 467.5 -> 359.2 mm, vias 1 -> 0
- net /~MEM_RD: track 241.5 -> 168.6 mm
- net /SLT2_SND: track 163.8 -> 91.5 mm
- net /Memory/~PAGE_RD: track 235.8 -> 164.0 mm
- net /Memory/~PAGE_WR: track 259.3 -> 187.7 mm
- net /Slots/SLT_DIR: track 202.8 -> 131.3 mm
- net /Slots/~CS1: track 193.0 -> 258.8 mm
- net VSS: track 337.5 -> 273.4 mm
- net /Slots/B_CLK: track 129.7 -> 66.5 mm, vias 1 -> 0
- net /D3: track 518.7 -> 457.7 mm
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Other:
- board text added: "Workaround: Keyboard Pull-ups"

Commit message: Mainboard: Update schematic and PCB layout with latest fixes
Signed-off-by: Sergey Kiselev <skiselev@gmail.com>
Parts:
- D1: value 1N4004 -> 1N4148
- U46: value ADM693 -> ADM691A
- U48: value OPA340P -> MCP601
- moved C59 27.9 mm to (109.2, 47.0), turned to 90 degrees
- moved R14 20.3 mm to (129.5, 47.0)
- moved C83 15.2 mm to (127.0, 47.0)
- moved C48 7.62 mm to (106.7, 47.0)
- moved R20 5.68 mm to (118.1, 58.4)
- moved R21 5.68 mm to (118.1, 55.9)
- moved U48 5.08 mm to (118.1, 47.0)
- moved Q1 1.27 mm to (135.9, 45.7)
Connections:
- U28 pad 10: /PSG/~RGT_B -> /PSG/~LFT_B
- U28 pad 11: /PSG/~RGT_A -> /PSG/~LFT_A
- U28 pad 12: /PSG/JOY_LFT -> /PSG/JOY_RGT
- U28 pad 13: /PSG/~LFT_B -> /PSG/~RGT_B
- U28 pad 14: /PSG/~LFT_A -> /PSG/~RGT_A
- U28 pad 9: /PSG/JOY_RGT -> /PSG/JOY_LFT
- U4 pad 18: /PSG/JOY_LFT -> /PSG/JOY_RGT
- U4 pad 19: /PSG/JOY_RGT -> /PSG/JOY_LFT
Routing:
- net GND: track 4713.7 -> 4731.0 mm
- net /PSG/~RGT_A: track 52.2 -> 37.6 mm
- net Net-(C83-Pad2): track 27.6 -> 17.9 mm
- net /PSG/~LFT_B: track 57.5 -> 66.6 mm
- net /PSG/~RGT_B: track 70.2 -> 61.6 mm
- net /PSG/~LFT_A: track 38.0 -> 45.0 mm
- net Net-(C59-Pad1): track 13.8 -> 20.4 mm
- net /PSG/JOY_RGT: track 70.6 -> 76.4 mm
- net /PSG/JOY_LFT: track 76.4 -> 70.6 mm
- net Net-(C83-Pad1): track 80.4 -> 75.1 mm
- net /CAS_IN: track 87.4 -> 84.4 mm
- net Net-(Q1-Pad2): track 15.6 -> 14.4 mm
- net Net-(D1-Pad2): track 23.5 -> 22.2 mm
- net VCC: track 2264.8 -> 2263.6 mm
- net /Processor/ALARM: track 173.2 -> 172.1 mm
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Other:
- board text added: "Keyboard pull-ups Populate only for Keyboard version 1.0"
- board text removed: "Workaround: Keyboard Pull-ups"

Commit message: Mainboard: Replace RGB and Cassette connectors with DIN8
Signed-off-by: Sergey Kiselev <skiselev@gmail.com>
Parts:
- removed the C51 at (33.0, 25.4)
- removed the C52 at (35.6, 25.4)
- removed the C57 at (96.5, 47.0)
- removed the C73 at (162.6, 34.5)
- removed the C80 at (167.6, 31.8)
- removed the C81 at (172.7, 21.6)
- removed the C94 at (33.0, 67.3)
- removed C95: 22pF, My_Components:Cap_Cer_508
- removed the R15 at (167.6, 55.9)
- removed the R17 at (170.2, 21.6)
- removed the R25 at (154.9, 34.3)
- removed the R33 at (149.9, 55.9)
- removed the R41 at (165.1, 21.6)
- removed the R42 at (63.5, 47.0)
- removed the R43 at (83.8, 47.0)
- removed the R48 at (63.5, 21.6)
- added C55: 0.1uF, My_Components:Cap_Cer_508, F.Cu at (91.4, 47.0)
- added C71: 10uF, My_Components:Cap_Elec_Radial_5mm, F.Cu at (160.0, 38.1)
- added C77: 10uF, My_Components:Cap_Elec_Radial_5mm, F.Cu at (83.8, 49.5)
- added C78: 1uF, My_Components:Cap_Elec_Radial_5mm, F.Cu at (147.3, 58.4)
- added C91: 27pF, My_Components:Cap_Cer_508, F.Cu at (73.7, 47.0)
- added C93: 22pF, My_Components:Cap_Cer_508, F.Cu at (33.0, 67.3)
- added R14: 10k, My_Components:Res_762, F.Cu at (63.5, 20.3)
- added R16: 4.7k, My_Components:Res_762, F.Cu at (130.8, 53.3)
- added R20: 4.7k, My_Components:Res_762, F.Cu at (167.6, 47.0)
- added R27: 2.7k, My_Components:Res_762, F.Cu at (165.1, 34.3)
- added R36: 1k, My_Components:Res_762, F.Cu at (66.0, 20.3)
- added R37: 470, My_Components:Res_762, F.Cu at (96.5, 47.0)
- added R38: 180, My_Components:Res_762, F.Cu at (38.1, 20.3)
- added R39: 120, My_Components:Res_762, F.Cu at (35.6, 20.3)
- added R45: 100, My_Components:Res_762, F.Cu at (139.7, 34.3)
- added R46: 75, My_Components:Res_762, F.Cu at (63.5, 47.0)
- added R47: 75, My_Components:Res_762, F.Cu at (78.7, 47.0)
- C79: value 10uF -> 22nF; footprint My_Components:Cap_Elec_Radial_5mm -> My_Components:Cap_Cer_508
- C89: renamed from C91; value 27pF -> 30pF
- C90: renamed from C92; value 27pF -> 30pF
- J5, J6: footprint My_Components:Conn_Mini_DIN_8pin -> My_Components:Conn_DIN_8pin
- R35: value 470 -> 1k
- moved C90 50.1 mm to (33.0, 72.4)
- moved D1 44.3 mm to (177.8, 20.3), turned to 270 degrees
- moved C79 43.3 mm to (132.1, 47.0), turned to 270 degrees
- moved R18 39.7 mm to (137.2, 47.0), turned to 90 degrees
- moved R17 36.9 mm to (130.8, 55.9)
- moved R35 35.6 mm to (134.6, 47.0)
- moved RY1 30.7 mm to (170.2, 20.3), turned to 90 degrees
- moved C58 25.4 mm to (88.9, 35.6)
- moved J2 25.4 mm to (76.2, 16.5)
- moved J4 25.4 mm to (101.6, 12.7)
- moved C75 22.9 mm to (154.9, 58.4)
- moved R19 20.3 mm to (137.2, 34.3), turned to 90 degrees
- moved C73 19.1 mm to (139.7, 58.4)
- moved R10 19.1 mm to (130.8, 58.4)
- moved R11 17.8 mm to (162.6, 47.0)
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- renumbered C53 to C51, C54 to C52, C55 to C53, C56 to C54, C58 to C56, C59 to C57, C60 to C58, C61 to C59, C62 to C60, C63 to C61, C64 to C62, C65 to C63, C66 to C64, C67 to C65, C68 to C66, C69 to C67, C70 to C68, C71 to C69, C72 to C70, C74 to C72, C75 to C73, C76 to C74, C77 to C75, C78 to C76, C82 to C80, C83 to C81, C84 to C82, C85 to C83, C86 to C84, C87 to C85, C88 to C86, C89 to C87, C90 to C88, C93 to C92, C96 to C94, R14 to R15, R16 to R17, R20 to R21, R21 to R22, R22 to R23, R23 to R24, R24 to R25, R27 to R28, R28 to R29, R29 to R30, R30 to R31, R31 to R32, R32 to R33, R36 to R40, R37 to R41, R38 to R42, R39 to R43, R40 to R44, R44 to R48, R45 to R49, R46 to R50, R47 to R51
Connections:
- C58 pad 2: Net-(C60-Pad2) -> /VDP/COMP
- C80 pad 1: Net-(C82-Pad1) -> Net-(C80-Pad1)
- C90 pad 1: Net-(C92-Pad1) -> GND
- C90 pad 2: Net-(C92-Pad2) (its old number) -> Net-(C90-Pad2)
- J2 pad 1: Net-(C60-Pad2) -> /VDP/COMP
- J5 pad 2: /VDP/LUMA -> /AUDIO
- J5 pad 3: /VDP/CHROMA -> /VDP/AV
- J5 pad 4: /VDP/GOUT -> /VDP/COMP
- J5 pad 5: /AUDIO -> /VDP/YS
- J5 pad 7: /VDP/BOUT -> /VDP/GOUT
- J5 pad 8: Net-(J5-Pad8) -> /VDP/BOUT
- J6 pad 1: Net-(J6-Pad1) -> GND
- J6 pad 2: Net-(J6-Pad2) -> GND
- J6 pad 4: GND -> Net-(J6-Pad4)
- J6 pad 5: GND -> Net-(C80-Pad1)
- J6 pad 6: Net-(C82-Pad1) -> Net-(J6-Pad6)
- J6 pad 7: GND -> Net-(J6-Pad7)
- J6 pad 8: Net-(J6-Pad8) -> GND
- L1 pad 1: Net-(C92-Pad2) (its old number) -> Net-(C91-Pad2)
- R12 pad 2: Net-(C73-Pad1) -> Net-(C71-Pad1)
- R18 pad 2: Net-(J6-Pad8) -> Net-(C79-Pad1)
- R19 pad 1: Net-(C73-Pad1) -> Net-(C79-Pad1)
- R19 pad 2: Net-(R19-Pad2) -> Net-(J6-Pad4)
- R26 pad 1: Net-(C73-Pad1) -> Net-(C71-Pad1)
- R26 pad 2: VCC -> GND
- R33 pad 1: Net-(C95-Pad2) -> Net-(C90-Pad2)
- R34 pad 1: /CAS_IN -> /CAS_MOT
- R34 pad 2: VCC -> Net-(Q1-Pad2)
- R35 pad 1: /PSG_SND -> /CAS_IN
- R35 pad 2: GND -> VCC
- R4 pad 1: Net-(R19-Pad2) -> Net-(R20-Pad2)
- RY1 pad 10: Net-(J6-Pad1) -> Net-(J6-Pad7)
- RY1 pad 5: Net-(J6-Pad2) -> Net-(J6-Pad6)
- RY1 pad 6: Net-(J6-Pad2) -> Net-(J6-Pad6)
- U47 pad 14: Net-(C79-Pad1) -> Net-(C77-Pad1)
- U47 pad 17: Net-(C92-Pad1) -> Net-(C91-Pad1)
- U49 pad 2: Net-(R19-Pad2) -> Net-(R20-Pad2)
- Y3 pad 2: Net-(C95-Pad2) -> Net-(C90-Pad2)
Routing:
- net VCC: track 2263.6 -> 2373.8 mm
- net Net-(C60-Pad2): track 59.8 -> 0.00 mm
- net /VDP/COMP: track 0.00 -> 52.5 mm
- net /VDP/CHROMA: track 61.0 -> 13.2 mm
- net Net-(J6-Pad6): track 0.00 -> 35.0 mm
- net Net-(C81-Pad1): track 75.1 -> 40.6 mm
- net Net-(R19-Pad2): track 33.3 -> 0.00 mm
- net /VDP/LUMA: track 41.7 -> 10.8 mm
- net Net-(C73-Pad1): track 27.1 -> 0.00 mm
- net Net-(C58-Pad1): track 54.5 -> 27.5 mm
- net /SLT2_SND: track 91.5 -> 116.4 mm
- net Net-(C82-Pad1): track 23.6 -> 0.00 mm
- net Net-(D1-Pad2): track 22.2 -> 45.7 mm
- net Net-(R20-Pad2): track 0.00 -> 22.4 mm
- net Net-(C74-Pad2): track 6.93 -> 29.0 mm
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Other:
- board text added: "0.5"
- board text added: "1.0"
- board text added: "2.0"
- board text added: "2.075"
- board text added: "5V Only"
- board text added: "Composite"
- board text removed: "Chroma"
- board text removed: "JP1 - Flash ROM A18 Select Open: A18=0 (default); Closed: A18=1"
- board text removed: "JP2: Japanese keyboard layout Open: JIS; Closed: ANSI/AIUEO/50on"
- board text removed: "JP3: 1-2: V9938; 2-3: V9958 (Use wire links instead of jumpers)"
- board text removed: "JP4, JP5: 1-2: NTSC; 2-3: PAL (Use wire links instead of jumpers)"
- board text removed: "Keyboard pull-ups Populate only for Keyboard version 1.0"
- board text removed: "Luma"
- board text removed: "Omega Home Computer Main Board - Version 1.1 Copyright (C) 2018-2019 Sergey Kiselev"
- board text removed: "PAL Clock Generator"
- board text removed: "Sync"
- board text removed: "[Chip Select]"
- board text removed: "[Slot Direction]"
- board text removed: "[Slot Select]"
- board text removed: "github.com/skiselev/omega www.malinov.com"
