File: Mainboard/KiCad/Omega-Mainboard.kicad_pcb (KiCad board)
At the start: 2 copper layers, 333.4 x 149.9 mm, 247 parts, among them J1 5V, J10 POWER, J11 KEYBOARD, J12 RAM_EXT, J13 ~RST~/~NMI, J14 CBUS, J2 Composite, J3 Audio, J4 S-VIDEO, J5 RGB, J6 Cassette, J7 JOYSTICK_A, J8 JOYSTICK_B, J9 PRINTER, Q1 PN2907A, Q2 PN2907A, U1 Z84C00, U10 D41464, U11 D41464, U12 ATF16V8B, U13 ATF16V8B, U14 ATF16V8B, U15 74HCT670, U16 74HCT670, U17 74HCT670, U18 74HCT670, U19 74F541, U2 82C55, U20 74F541, U21 74F541, U22 74HCT540, U23 74HCT273, U24 74HCT273, U25 74F245, U26 74F245, U27 74HCT175, U28 74HCT157, U29 74HCT157, U3 V9938, U30 74HCT153, U31 74HCT153, U32 74AHCT138, U33 74AHCT125, U34 74HCT74, U35 74HCT74, U36 74HCT74, U37 74AHCT32, U38 74AHCT32, U39 74AHCT32, U4 YM2149, U40 74HCT30, U41 74HCT30, U42 74LS07, U43 74HCT04, U44 74AHCT02, U45 74HCT00, U46 ADM691A, U47 CXA1645, U48 MCP601, U49 LM311, U5 RP5C01, U6 SST39SF040, U7 AS6C4008, U8 D41464, U9 D41464, Y1 21.477270MHz, Y2 32768 Hz, Y3 4.433618MHz

Commit message: Mainboard: Final v1.1 design files
Signed-off-by: Sergey Kiselev <skiselev@gmail.com>
Parts:
- added JP4: V9938/V9958, My_Components:Conn_Pin_Header_3x1_2.54mm, F.Cu at (40.6, 63.5)
- C65, C66, C67: value 47uF -> 100uF
- C68, C69, C70: footprint My_Components:Cap_Elec_Radial_5mm -> My_Components:Cap_Pol_508_3
- J14: footprint My_Components:Conn_Pin_Header_11x1_2.54mm -> My_Components:Conn_Pin_Header_13x1_2.54mm
- U3: value V9938 -> V9938/V9958
- U48: value MCP601 -> MCP6281
- moved C47 5.08 mm to (81.3, 73.7)
- moved C69 3.81 mm to (77.5, 73.7), turned to 90 degrees
- moved J14 1.31 mm to (77.2, 121.9)
- moved C68 1.27 mm to (307.3, 124.5)
- moved C70 1.27 mm to (55.9, 152.4)
- moved C74 0.63 mm to (154.9, 58.4)
- renumbered JP4 to JP5, JP5 to JP6
Connections:
- J14 pad 10: /VDP/CB0 -> /VDP/CB2
- J14 pad 11: GND -> /VDP/CB1
- J14 pad 2: /VDP/CBDR -> /VDP/~DHCLK
- J14 pad 3: /VDP/CB7 -> /VDP/~DLCLK
- J14 pad 4: /VDP/CB6 -> /VDP/CBDR
- J14 pad 5: /VDP/CB5 -> /VDP/CB7
- J14 pad 6: /VDP/CB4 -> /VDP/CB6
- J14 pad 7: /VDP/CB3 -> /VDP/CB5
- J14 pad 8: /VDP/CB2 -> /VDP/CB4
- J14 pad 9: /VDP/CB1 -> /VDP/CB3
- RR3 pad 2: Net-(RR3-Pad2) -> /VDP/~DHCLK
- RR3 pad 3: Net-(RR3-Pad3) -> /VDP/~DLCLK
- U3 pad 2: Net-(RR3-Pad2) -> /VDP/~DHCLK
- U3 pad 3: Net-(RR3-Pad3) -> /VDP/~DLCLK
- U43 pad 6: /VDP/SYNCIN -> Net-(JP4-Pad1)
Routing:
- net /VDP/~DLCLK: track 0.00 -> 17.8 mm
- net /VDP/~DHCLK: track 0.00 -> 17.5 mm
- net Net-(JP4-Pad1): track 0.00 -> 9.72 mm
- net Net-(RR3-Pad3): track 8.73 -> 0.00 mm
- net /VDP/SYNCIN: track 52.0 -> 43.3 mm
- net Net-(RR3-Pad2): track 8.41 -> 0.00 mm
- net Net-(JP4-Pad3): track 5.08 -> 10.2 mm
- net /VDP/PAL_CLK: track 58.6 -> 54.9 mm
- net VCCRGB: track 50.2 -> 47.5 mm
- net GND: track 4875.1 -> 4876.4 mm, vias 46 -> 48
- net VCCVDP: track 86.9 -> 85.7 mm
- net VCC: track 2306.1 -> 2305.0 mm
- net /Memory/RAM_A15: track 106.5 -> 106.0 mm
Other:
- board text added: "JP3, JP4: 1-2: V9938; 2-3: V9958 (Use wire links instead of jumpers)"
- board text added: "JP5, JP6: 1-2: NTSC; 2-3: PAL (Use wire links instead of jumpers)"
- board text added: "Omega Home Computer - Main Board - Version 1.1 Copyright (C) 2018-2019 Sergey Kiselev"
- board text added: "~NMI"
- board text added: "~RST"
- board text removed: "JP3: 1-2: V9938; 2-3: V9958 (Use wire links instead of jumpers)"
- board text removed: "JP4, JP5: 1-2: NTSC; 2-3: PAL (Use wire links instead of jumpers)"
- board text removed: "Omega Home Computer Main Board - Version 1.1 Copyright (C) 2018-2019 Sergey Kiselev"

Commit message: Mainboard: Update to version 1.2
Signed-off-by: Sergey Kiselev <skiselev@gmail.com>
Parts:
- L2, L3: value 5.7uH -> 5.6uH
- R30: value 1K -> 1k
Other:
- board text added: "Omega Home Computer - Main Board - Version 1.2 Copyright (C) 2018-2020 Sergey Kiselev"
- board text removed: "Omega Home Computer - Main Board - Version 1.1 Copyright (C) 2018-2019 Sergey Kiselev"
Changed lines of the file:
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@@
       (effects (font (size 1.016 1.016) (thickness 0.2032)))
     )
-    (fp_text value 5.7uH (at -5.3975 0.3175) (layer F.SilkS)
+    (fp_text value 5.6uH (at -5.3975 0.3175) (layer F.SilkS)
       (effects (font (size 1.016 0.9144) (thickness 0.2032) italic))
     )
@@
       (effects (font (size 1.016 1.016) (thickness 0.2032)))
     )
-    (fp_text value 5.7uH (at 1.5875 -1.905 90) (layer F.SilkS)
+    (fp_text value 5.6uH (at 1.5875 -1.905 90) (layer F.SilkS)
       (effects (font (size 1.016 0.9144) (thickness 0.2032) italic))
     )
@@
       (effects (font (size 1.016 1.016) (thickness 0.2032)))
     )
-    (fp_text value 1K (at -6.0325 0.3175 90) (layer F.SilkS)
+    (fp_text value 1k (at -6.0325 0.3175 90) (layer F.SilkS)
       (effects (font (size 1.016 0.9144) (thickness 0.2032) italic))
     )
@@
     (effects (font (size 1 1) (thickness 0.15)) (justify left))
   )
-  (gr_text "Omega Home Computer - Main Board - Version 1.1\nCopyright (C) 2018-2019 Sergey Kiselev" (at 288.29 58.42) (layer F.SilkS)
+  (gr_text "Omega Home Computer - Main Board - Version 1.2\nCopyright (C) 2018-2020 Sergey Kiselev" (at 288.29 58.42) (layer F.SilkS)
     (effects (font (size 1.5 1.5) (thickness 0.3)))
   )

Commit message: Add files for version 1.3eu from Jordi Solis
Signed-off-by: Sergey Kiselev <skiselev@gmail.com>
Parts:
- added JP10: 4Mb, Connector_PinHeader_2.54mm:PinHeader_1x02_P2.54mm_Vertical, F.Cu at (273.8, 96.5)
- added JP11: 2Mb, Connector_PinHeader_2.54mm:PinHeader_1x02_P2.54mm_Vertical, F.Cu at (276.4, 96.5)
- added JP12: 1Mb, Connector_PinHeader_2.54mm:PinHeader_1x02_P2.54mm_Vertical, F.Cu at (278.9, 96.5)
- added JP7: 1Mb, Connector_PinHeader_2.54mm:PinHeader_1x03_P2.54mm_Vertical, F.Cu at (317.1, 139.7)
- added JP8: 2Mb, Connector_PinHeader_2.54mm:PinHeader_1x03_P2.54mm_Vertical, F.Cu at (319.7, 139.7)
- added JP9: 4Mb, Connector_PinHeader_2.54mm:PinHeader_1x03_P2.54mm_Vertical, F.Cu at (322.2, 139.7)
- added RR10: 4.7k, Resistor_THT:R_Array_SIP6, F.Cu at (314.5, 156.2)
- J5, J6: footprint My_Components:Conn_DIN_8pin -> artemisa:DIN8
- JP4: footprint My_Components:Conn_Pin_Header_3x1_2.54mm -> artemisa:Conn_Pin_Header_3x1_2.54mm
- moved U15 3.94 mm to (255.3, 98.9)
- moved C15 3.81 mm to (241.3, 99.1)
- moved JP4 0.13 mm to (40.6, 63.4)
- turned J5 to 180 degrees
- turned J6 to 180 degrees
- turned R13 to 180 degrees
Connections:
- J4 pad ~: GND -> (no net)
- J7 pad GND: GND -> (no net)
- J8 pad GND: GND -> (no net)
- J9 pad GND: GND -> (no net)
- R13 pad 1: /Memory/ROM_A18 -> GND
- R13 pad 2: GND -> /Memory/ROM_A18
- U15 pad 10: /D6 -> Net-(JP11-Pad2)
- U15 pad 7: /D5 -> Net-(JP12-Pad2)
- U15 pad 9: /D7 -> Net-(JP10-Pad2)
- U32 pad 1: /Memory/RAM_A19 -> Net-(JP7-Pad2)
- U32 pad 2: /Memory/RAM_A20 -> Net-(JP8-Pad2)
- U32 pad 3: /Memory/RAM_A21 -> Net-(JP9-Pad2)
- Y2 pad ~: GND -> (no net)
Routing:
- net /VDP/COMP: track 52.5 -> 81.5 mm
- net Net-(JP12-Pad2): track 0.00 -> 26.5 mm
- net Net-(JP7-Pad2): track 0.00 -> 23.3 mm
- net Net-(JP8-Pad2): track 0.00 -> 19.5 mm
- net /Memory/RAM_A19: track 87.5 -> 69.2 mm
- net /D5: track 360.0 -> 378.2 mm, vias 0 -> 1
- net Net-(JP11-Pad2): track 0.00 -> 16.5 mm
- net /Memory/RAM_A20: track 91.2 -> 75.0 mm
- net /D6: track 352.7 -> 367.8 mm
- net VCC: track 2305.0 -> 2319.1 mm
- net /Memory/RAM_A21: track 87.7 -> 74.2 mm
- net Net-(JP9-Pad2): track 0.00 -> 12.5 mm
- net Net-(JP9-Pad3): track 0.00 -> 11.5 mm
- net Net-(JP8-Pad3): track 0.00 -> 11.5 mm
- net Net-(JP7-Pad3): track 0.00 -> 11.5 mm
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Other:
- outline, holes or cut-outs redrawn
- board text added: "Omega Home Computer - Main Board - Version 1.3 eu (msxmakers) Copyright (C) 2018-2020 Sergey Kiselev"
- board text removed: "Omega Home Computer - Main Board - Version 1.2 Copyright (C) 2018-2020 Sergey Kiselev"

Commit message: Version 1.4: Add cut-out for the right angle slot connector. Add optional jumpers to limit memory mapper address range
Signed-off-by: Sergey Kiselev <skiselev@gmail.com>
Parts:
- removed JP10: 4Mb, Connector_PinHeader_2.54mm:PinHeader_1x02_P2.54mm_Vertical
- removed JP11: 2Mb, Connector_PinHeader_2.54mm:PinHeader_1x02_P2.54mm_Vertical
- removed JP12: 1Mb, Connector_PinHeader_2.54mm:PinHeader_1x02_P2.54mm_Vertical
- removed JP9: 4Mb, Connector_PinHeader_2.54mm:PinHeader_1x03_P2.54mm_Vertical
- removed REF**: OSHW-Logo_7.5x8mm_SilkScreen, Symbol:OSHW-Logo_7.5x8mm_SilkScreen
- removed REF**: KiCad-Logo2_5mm_SilkScreen, Symbol:KiCad-Logo2_5mm_SilkScreen
- removed ~: Symbol_GNU-Logo_SilkscreenTop, Symbol:Symbol_GNU-Logo_SilkscreenTop
- J5, J6: footprint artemisa:DIN8 -> My_Components:Conn_DIN_8pin
- JP4: footprint artemisa:Conn_Pin_Header_3x1_2.54mm -> My_Components:Conn_Pin_Header_3x1_2.54mm
- JP7: value 1Mb -> RAM_SIZE; footprint Connector_PinHeader_2.54mm:PinHeader_1x03_P2.54mm_Vertical -> My_Components:Conn_Pin_Header_2x3_2.54mm
- JP8: value 2Mb -> RAM_SIZE; footprint Connector_PinHeader_2.54mm:PinHeader_1x03_P2.54mm_Vertical -> My_Components:Conn_Pin_Header_2x3_2.54mm
- RR10: footprint Resistor_THT:R_Array_SIP6 -> My_Components:Conn_SIL6
- moved JP8 62.6 mm to (275.6, 95.2)
- moved RR10 25.8 mm to (335.3, 141.0), turned to 90 degrees
- moved U15 3.94 mm to (255.3, 102.9)
- moved C15 3.81 mm to (241.3, 102.9)
- moved JP7 3.15 mm to (320.0, 141.0)
- moved JP4 0.13 mm to (40.6, 63.5)
- turned J5 to 0 degrees
- turned J6 to 0 degrees
- turned R13 to 0 degrees
Connections:
- J4 pad ~: (no net) -> GND
- J7 pad GND: (no net) -> GND
- J8 pad GND: (no net) -> GND
- J9 pad GND: (no net) -> GND
- JP7 pad 2: Net-(JP7-Pad2) -> /Memory/RAM_A19
- JP7 pad 3: Net-(JP7-Pad3) -> /Memory/RAM_A20
- JP8 pad 1: /Memory/RAM_A20 -> /D6
- JP8 pad 2: Net-(JP8-Pad2) -> /D6
- JP8 pad 3: Net-(JP8-Pad3) -> /D7
- R13 pad 1: GND -> /Memory/ROM_A18
- R13 pad 2: /Memory/ROM_A18 -> GND
- RR10 pad 2: Net-(JP7-Pad3) -> /Memory/RAM_A19
- RR10 pad 3: Net-(JP8-Pad3) -> /Memory/RAM_A20
- RR10 pad 4: Net-(JP9-Pad3) -> /Memory/RAM_A21
- U15 pad 10: Net-(JP11-Pad2) -> /D6
- U15 pad 7: Net-(JP12-Pad2) -> /D5
- U15 pad 9: Net-(JP10-Pad2) -> /D7
- U32 pad 1: Net-(JP7-Pad2) -> /Memory/RAM_A19
- U32 pad 2: Net-(JP8-Pad2) -> /Memory/RAM_A20
- U32 pad 3: Net-(JP9-Pad2) -> /Memory/RAM_A21
- Y2 pad ~: (no net) -> GND
Routing:
- net /VDP/COMP: track 81.5 -> 52.5 mm
- net /Memory/RAM_A19: track 69.2 -> 95.9 mm
- net Net-(JP12-Pad2): track 26.5 -> 0.00 mm
- net /D5: track 378.2 -> 404.0 mm, vias 1 -> 2
- net /Memory/RAM_A20: track 75.0 -> 99.5 mm
- net Net-(JP7-Pad2): track 23.3 -> 0.00 mm
- net /Memory/RAM_A21: track 74.2 -> 94.8 mm
- net Net-(JP8-Pad2): track 19.5 -> 0.00 mm
- net /D7: track 332.7 -> 352.0 mm
- net Net-(JP11-Pad2): track 16.5 -> 0.00 mm
- net GND: track 4878.6 -> 4894.1 mm
- net VCC: track 2319.1 -> 2305.9 mm
- net /D6: track 367.8 -> 380.7 mm
- net Net-(JP9-Pad2): track 12.5 -> 0.00 mm
- net Net-(JP9-Pad3): track 11.5 -> 0.00 mm
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Other:
- board text added: "1MB"
- board text added: "2MB"
- board text added: "4MB"
- board text added: "Omega Home Computer - Main Board - Version 1.4 Copyright (C) 2018-2021 Sergey Kiselev"
- board text removed: "Omega Home Computer - Main Board - Version 1.3 eu (msxmakers) Copyright (C) 2018-2020 Sergey Kiselev"
