File: Mainboard/KiCad/Omega-Processor.sch (KiCad schematic (older format))
At the start: 24 parts, among them J9 PRINTER, U1 Z84C00, U12 ATF16V8B, U24 74HCT273, U27 74HCT175, U33 74AHCT125, U34 74HCT74, U35 74HCT74, U37 74AHCT32, U42 74LS07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

Commit message: Mainboard: Replace RGB and Cassette connectors with DIN8
Signed-off-by: Sergey Kiselev <skiselev@gmail.com>
Parts:
- renumbered C87 to C85, C89 to C87, C90 to C88, R31 to R32
Changed lines of the file:
@@
 $EndComp
 $Comp
-L Device:C C87
+L Device:C C85
 U 1 1 5BF85069
 P 7750 3800
-F 0 "C87" H 7775 3900 50  0000 L CNN
+F 0 "C85" H 7775 3900 50  0000 L CNN
 F 1 "68pF" H 7775 3700 50  0000 L CNN
 F 2 "My_Components:Cap_Cer_508" H 7788 3650 50  0001 C CNN
@@
 $EndComp
 $Comp
-L Device:C C90
+L Device:C C88
 U 1 1 5BF850EC
 P 7750 4300
-F 0 "C90" H 7775 4400 50  0000 L CNN
+F 0 "C88" H 7775 4400 50  0000 L CNN
 F 1 "33pF" H 7775 4200 50  0000 L CNN
 F 2 "My_Components:Cap_Cer_508" H 7788 4150 50  0001 C CNN
@@
 $EndComp
 $Comp
-L Device:C C89
+L Device:C C87
 U 1 1 5BF8514D
 P 7750 4800
-F 0 "C89" H 7775 4900 50  0000 L CNN
+F 0 "C87" H 7775 4900 50  0000 L CNN
 F 1 "33pF" H 7775 4700 50  0000 L CNN
 F 2 "My_Components:Cap_Cer_508" H 7788 4650 50  0001 C CNN
@@
 Connection ~ 3900 2900
 $Comp
-L Device:R R31
+L Device:R R32
 U 1 1 5C039811
 P 900 1750
-F 0 "R31" V 980 1750 50  0000 C CNN
+F 0 "R32" V 980 1750 50  0000 C CNN
 F 1 "1k" V 900 1750 50  0000 C CNN
 F 2 "My_Components:Res_762" V 830 1750 50  0001 C CNN
