File: Mainboard/KiCad/Omega-PPI.sch (KiCad schematic (older format))
At the start: 14 parts, among them J11 KEYBOARD, U13 ATF16V8B, U2 82C55, U22 74HCT540, U23 74HCT273, U30 74HCT153, U31 74HCT153, U38 74AHCT32, U40 74HCT30, U41 74HCT30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

Commit message: Mainboard: Fix some of the issues described in #1
Signed-off-by: Sergey Kiselev <skiselev@gmail.com>
Parts:
- removed R22, R23, R24: 4.7k, My_Components:Res_762, symbol Device:R
- added RR7: 4.7k, My_Components:Conn_SIL10, symbol my_components:RR9
Connections:
- net COLUMN0: now also RR7.2
- net COLUMN1: now also RR7.3
- net COLUMN2: now also RR7.4
- net COLUMN3: now also RR7.5
- net COLUMN4: now also RR7.6
- net COLUMN5: now also RR7.7
- net COLUMN6: now also RR7.8
- net COLUMN7: now also RR7.9
- net VCC: now also RR7.1 (COM)
- new net PRT_BUSY: RR7.10
Other:
- note added: "Keyboard Pull-ups"
- note removed: "Keyboard Pull-ups Errata Workaround"
Changed lines of the file:
@@
 Wire Wire Line
 	3300 5650 3300 7500
-$Comp
-L Device:R R22
-U 1 1 5F651789
-P 9650 5600
-F 0 "R22" V 9550 5500 50  0000 C CNN
-F 1 "4.7k" V 9550 5700 50  0000 C CNN
-F 2 "My_Components:Res_762" V 9580 5600 50  0001 C CNN
-F 3 "~" H 9650 5600 50  0001 C CNN
-	1    9650 5600
-	0    1    1    0
-$EndComp
-$Comp
-L Device:R R23
-U 1 1 5F651EB8
-P 9650 5800
-F 0 "R23" V 9550 5700 50  0000 C CNN
-F 1 "4.7k" V 9550 5900 50  0000 C CNN
-F 2 "My_Components:Res_762" V 9580 5800 50  0001 C CNN
-F 3 "~" H 9650 5800 50  0001 C CNN
-	1    9650 5800
-	0    1    1    0
-$EndComp
-$Comp
-L Device:R R24
-U 1 1 5F652358
-P 9650 6000
-F 0 "R24" V 9550 5900 50  0000 C CNN
-F 1 "4.7k" V 9550 6100 50  0000 C CNN
-F 2 "My_Components:Res_762" V 9580 6000 50  0001 C CNN
-F 3 "~" H 9650 6000 50  0001 C CNN
-	1    9650 6000
-	0    1    1    0
-$EndComp
 Wire Wire Line
-	9500 5600 9000 5600
+	10000 5300 9500 5300
 Wire Wire Line
-	9500 5800 9000 5800
+	10000 5500 9500 5500
 Wire Wire Line
-	9500 6000 9000 6000
+	10000 5700 9500 5700
 Wire Wire Line
-	9800 5600 10000 5600
-Wire Wire Line
-	10000 5600 10000 5500
-Wire Wire Line
-	9800 5800 10000 5800
-Wire Wire Line
-	10000 5800 10000 5600
-Connection ~ 10000 5600
-Wire Wire Line
-	9800 6000 10000 6000
-Wire Wire Line
-	10000 6000 10000 5800
-Connection ~ 10000 5800
+	9900 5200 9900 5100
 $Comp
 L power:VCC #PWR02
 U 1 1 5F6C2774
-P 10000 5500
-F 0 "#PWR02" H 10000 5350 50  0001 C CNN
-F 1 "VCC" H 10017 5673 50  0000 C CNN
-F 2 "" H 10000 5500 50  0001 C CNN
-F 3 "" H 10000 5500 50  0001 C CNN
-	1    10000 5500
+P 9900 5100
+F 0 "#PWR02" H 9900 4950 50  0001 C CNN
+F 1 "VCC" H 9917 5273 50  0000 C CNN
+F 2 "" H 9900 5100 50  0001 C CNN
+F 3 "" H 9900 5100 50  0001 C CNN
+	1    9900 5100
 	1    0    0    -1
 $EndComp
-Text Label 9000 5600 0    60   ~ 0
+Text Label 9500 5300 0    60   ~ 0
 COLUMN0
-Text Label 9000 5800 0    60   ~ 0
+Text Label 9500 5500 0    60   ~ 0
 COLUMN2
-Text Label 9000 6000 0    60   ~ 0
+Text Label 9500 5700 0    60   ~ 0
 COLUMN4
-Text Notes 8600 5150 0    60   ~ 0
-Keyboard Pull-ups Errata Workaround
-Wire Notes Line
-	8500 5000 10500 5000
-Wire Notes Line
-	10500 5000 10500 6200
-Wire Notes Line
-	10500 6200 8500 6200
-Wire Notes Line
-	8500 6200 8500 5000
+Text Notes 10350 4800 2    60   ~ 0
+Keyboard Pull-ups
+$Comp
+L my_components:RR9 RR7
+U 1 1 5DB840FB
+P 10300 5650
+F 0 "RR7" H 10428 5686 50  0000 L CNN
+F 1 "4.7k" H 10428 5595 50  0000 L CNN
+F 2 "My_Components:Conn_SIL10" H 10300 5650 50  0001 C CNN
+F 3 "" H 10300 5650 50  0000 C CNN
+	1    10300 5650
+	1    0    0    -1
+$EndComp
+Wire Wire Line
+	9900 5200 10000 5200
+Wire Wire Line
+	10000 5400 9500 5400
+Wire Wire Line
+	10000 5600 9500 5600
+Wire Wire Line
+	10000 5800 9500 5800
+Wire Wire Line
+	10000 5900 9500 5900
+Wire Wire Line
+	10000 6000 9500 6000
+Text Label 9500 5400 0    60   ~ 0
+COLUMN1
+Text Label 9500 5600 0    60   ~ 0
+COLUMN3
+Text Label 9500 5800 0    60   ~ 0
+COLUMN5
+Text Label 9500 5900 0    60   ~ 0
+COLUMN6
+Text Label 9500 6000 0    60   ~ 0
+COLUMN7
+Text HLabel 10600 3600 2    60   Input ~ 0
+PRT_BUSY
+Wire Wire Line
+	10600 3600 10200 3600
+Text Label 10200 3600 0    60   ~ 0
+PRT_BUSY
+Wire Wire Line
+	10000 6100 9500 6100
+Text Label 9500 6100 0    60   ~ 0
+PRT_BUSY
 $EndSCHEMATC
