File: Mainboard/KiCad/Omega-VDP.sch (KiCad schematic (older format))
At the start: 63 parts, among them J2 Composite, J4 S-VIDEO, J5 RGB, Q2 PN2907A, U10 D41464, U11 D41464, U3 V9938, U39 74AHCT32, U43 74HCT04, U47 CXA1645, U8 D41464, U9 D41464, Y1 21.477270MHz, Y3 4.433618MHz

Commit message: Mainboard: Fix some of the issues described in #1
Signed-off-by: Sergey Kiselev <skiselev@gmail.com>
Parts:
- removed J5: RGB, My_Components:Conn_Mini_DIN_8pin, symbol Connector:Mini-DIN-8
- added J5: RGB, My_Components:Conn_DIN_8pin, symbol Connector:DIN-8
- added R14: 10k, My_Components:Res_762, symbol Device:R
- added R35: 180, My_Components:Res_762, symbol Device:R
- added R36: 120, My_Components:Res_762, symbol Device:R
- C89: renamed from C91; value 27pF -> 30pF
- C90: renamed from C92; value 27pF -> 30pF
- C91: renamed from C95; value 22pF -> 27pF
- R33: renamed from R48; value 0 -> 1k
- renumbered C53 to C51, C54 to C52, C55 to C53, C56 to C54, C57 to C55, C58 to C56, C60 to C59, C61 to C60, C62 to C61, C63 to C62, C64 to C63, C65 to C64, C79 to C77, C84 to C82, C85 to C83, C86 to C84, C88 to C86, C93 to C92, C94 to C93, C96 to C94, R27 to R25, R29 to R27, R30 to R28, R32 to R30, R36 to R37, R37 to R38, R38 to R39, R39 to R40, R42 to R43, R43 to R44, R44 to R45, R45 to R46, R46 to R47, R47 to R48, RR8 to RR9
Connections:
- net AUDIO: now also J5.2
- net BOUT: now also J5.8
- net GND: now also C90.1, U3.1 (GND), U3.20 (GND), U47.1 (GND), U47.24 (GND), J5.1, R14.1, R35.1; no longer C91.1
- net GOUT: now also J5.7
- net ROUT: now also J5.6
- net VCC: now also R33.2, R36.2; no longer JP3.3, JP4.1
- net VCCVDP: now reaches U3.58 (VCC)
- net VCCVDP: now also JP3.3
- net COMP: now reaches C59.2, J2.1 (In)
- net COMP: now also J5.4; no longer R33.1
- net VCCRGB: now reaches U47.12 (VCC)
- net VCCRGB: now also JP4.1, U47.19 (VCC)
- net at U47.17 (YTRAP): now also C91.1; no longer C90.1
- net at L1.1: now also C91.2; no longer C90.2
- net at R30.1, Y3.2: now also C90.2; no longer C91.2
- new net AV: J5.3, R14.2, R33.1
- new net YS: J5.5, R35.2, R36.1
Other:
- note added: "PAL: R9 - 16k, C91 - 18pF\nR9 - Tolerance 1%"
- note removed: "PAL: R9 - 16k, C92 - 18pF\nR9 - Tolerance 1%"
- moved on the sheet: C62, C63, C64, C90, C91, J2, JP4, R33, R37, R38, R39, R40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
