File: Mainboard/KiCad/Omega-Memory.sch (KiCad schematic (older format))
At the start: 12 parts, among them J12 RAM_EXT, U15 74HCT670, U16 74HCT670, U17 74HCT670, U18 74HCT670, U26 74F245, U32 74AHCT138, U37 74AHCT32, U6 SST39SF040, U7 AS6C4008

Commit message: Mainboard: Fix the issues discovered so far
Signed-off-by: Sergey Kiselev <skiselev@gmail.com>
Other:
- moved on the sheet: U37A, U37D
Changed lines of the file:
@@
 $Comp
 L my_components:74LS32 U37
-U 1 2 5BEFC84C
+U 4 2 5BEFC853
 P 1400 4550
 F 0 "U37" H 1400 4550 60  0000 C CNN
@@
 F 2 "My_Components:IC_DIP14_300" H 1400 4550 60  0001 C CNN
 F 3 "" H 1400 4550 60  0000 C CNN
-	1    1400 4550
-	1    0    0    -1
-$EndComp
-$Comp
-L my_components:74LS32 U37
-U 4 2 5BEFC853
-P 1400 4150
-F 0 "U37" H 1400 4150 60  0000 C CNN
-F 1 "74AHCT32" H 1300 4000 60  0000 L CNN
-F 2 "My_Components:IC_DIP14_300" H 1400 4150 60  0001 C CNN
-F 3 "" H 1400 4150 60  0000 C CNN
-	4    1400 4150
+	4    1400 4550
 	1    0    0    -1
 $EndComp
@@
 Wire Wire Line
 	1000 5650 1100 5650
+$Comp
+L my_components:74LS32 U37
+U 1 2 5BEFC84C
+P 1400 4150
+F 0 "U37" H 1400 4150 60  0000 C CNN
+F 1 "74AHCT32" H 1300 4000 60  0000 L CNN
+F 2 "My_Components:IC_DIP14_300" H 1400 4150 60  0001 C CNN
+F 3 "" H 1400 4150 60  0000 C CNN
+	1    1400 4150
+	1    0    0    -1
+$EndComp
 $EndSCHEMATC

Commit message: Mainboard: Fix some of the issues described in #1
Signed-off-by: Sergey Kiselev <skiselev@gmail.com>
Parts:
- U15, U16, U17, U18: symbol my_components:74LS670 -> 74xx:74LS670
- U26: symbol my_components:74LS245 -> 74xx:74LS245
- U32: symbol my_components:74LS138 -> 74xx:74LS138
- U6: symbol Omega-Mainboard-rescue:SST39SF040-my_components -> my_components:SST39SF040
- U7: symbol Omega-Mainboard-rescue:AS6C4008-my_components -> my_components:AS6C4008
Connections:
- wire segments 245 -> 261
Other:
- moved on the sheet: J12, JP1, R13, U15, U16, U17, U18, U37A, U37D, U6, U7

Commit message: Add files for version 1.3eu from Jordi Solis
Signed-off-by: Sergey Kiselev <skiselev@gmail.com>
Parts:
- added JP10: 4Mb, Connector_PinHeader_2.54mm:PinHeader_1x02_P2.54mm_Vertical, symbol Connector_Generic:Conn_01x02
- added JP11: 2Mb, Connector_PinHeader_2.54mm:PinHeader_1x02_P2.54mm_Vertical, symbol Connector_Generic:Conn_01x02
- added JP12: 1Mb, Connector_PinHeader_2.54mm:PinHeader_1x02_P2.54mm_Vertical, symbol Connector_Generic:Conn_01x02
- added JP7: 1Mb, Connector_PinHeader_2.54mm:PinHeader_1x03_P2.54mm_Vertical, symbol Connector_Generic:Conn_01x03
- added JP8: 2Mb, Connector_PinHeader_2.54mm:PinHeader_1x03_P2.54mm_Vertical, symbol Connector_Generic:Conn_01x03
- added JP9: 4Mb, Connector_PinHeader_2.54mm:PinHeader_1x03_P2.54mm_Vertical, symbol Connector_Generic:Conn_01x03
- added RR10: 4.7k, Resistor_THT:R_Array_SIP6, symbol Omega-Mainboard-rescue:RR5-my_components
- U37: symbol my_components:74LS32 -> Omega-Mainboard-rescue:74LS32-my_components
- U6: symbol my_components:SST39SF040 -> Omega-Mainboard-rescue:SST39SF040-my_components
- U7: symbol my_components:AS6C4008 -> Omega-Mainboard-rescue:AS6C4008-my_components
Connections:
- wire segments 261 -> 282
- no-connect marks 0 -> 2
Other:
- moved on the sheet: J12, JP1, R13, U16, U26, U32, U37A, U37D, U6, U7

Commit message: Version 1.4: Add cut-out for the right angle slot connector. Add optional jumpers to limit memory mapper address range
Signed-off-by: Sergey Kiselev <skiselev@gmail.com>
Parts:
- removed JP10: 4Mb, Connector_PinHeader_2.54mm:PinHeader_1x02_P2.54mm_Vertical, symbol Connector_Generic:Conn_01x02
- removed JP11: 2Mb, Connector_PinHeader_2.54mm:PinHeader_1x02_P2.54mm_Vertical, symbol Connector_Generic:Conn_01x02
- removed JP12: 1Mb, Connector_PinHeader_2.54mm:PinHeader_1x02_P2.54mm_Vertical, symbol Connector_Generic:Conn_01x02
- removed JP7: 1Mb, Connector_PinHeader_2.54mm:PinHeader_1x03_P2.54mm_Vertical, symbol Connector_Generic:Conn_01x03
- removed JP8: 2Mb, Connector_PinHeader_2.54mm:PinHeader_1x03_P2.54mm_Vertical, symbol Connector_Generic:Conn_01x03
- removed JP9: 4Mb, Connector_PinHeader_2.54mm:PinHeader_1x03_P2.54mm_Vertical, symbol Connector_Generic:Conn_01x03
- removed RR10: 4.7k, Resistor_THT:R_Array_SIP6, symbol Omega-Mainboard-rescue:RR5-my_components
- added JP7, JP8: RAM_SIZE, My_Components:Conn_Pin_Header_2x3_2.54mm, symbol Connector_Generic:Conn_02x03_Odd_Even
- added RR10: 4.7k, My_Components:Conn_SIL6, symbol my_components:RR5
- U37: symbol Omega-Mainboard-rescue:74LS32-my_components -> my_components:74LS32
- U7: symbol Omega-Mainboard-rescue:AS6C4008-my_components -> my_components:AS6C4008
Connections:
- wire segments 282 -> 280
Other:
- moved on the sheet: J12, JP1, R13, U16, U18, U26, U32, U37A, U37D, U6, U7

Commit message: Fix issue #56, where joystick A trigger 2 was swapped with joystick B trigger 1
Signed-off-by: Sergey Kiselev <skiselev@gmail.com>
Parts:
- U6: symbol Omega-Mainboard-rescue:SST39SF040-my_components -> my_components:SST39SF040
Connections:
- net GND: no longer U6.16 (GND), U7.16 (GND)
- net VCC: no longer U6.32 (VCC), U7.32 (VCC)
Changed lines of the file:
@@
 AR Path="/5BEB180B" Ref="U7"  Part="1"
 AR Path="/5BD9D8C5/5BEB180B" Ref="U7"  Part="1"
-F 0 "U7" H 5900 3700 60  0000 C CNN
-F 1 "AS6C4008" H 5900 3600 60  0000 C CNN
+F 0 "U7" H 5900 3650 60  0000 C CNN
+F 1 "AS6C4008" H 5900 3550 60  0000 C CNN
 F 2 "My_Components:IC_DIP32_600" H 6300 2300 60  0001 C CNN
 F 3 "" H 6300 2300 60  0000 C CNN
@@
 RAM_A18
 $Comp
-L Omega-Mainboard-rescue:SST39SF040-my_components U6
+L my_components:SST39SF040 U6
 U 1 1 5BEB1F99
 P 6300 5800
-F 0 "U6" H 5900 7200 60  0000 C CNN
-F 1 "SST39SF040" H 5900 7100 60  0000 C CNN
+F 0 "U6" H 5900 7150 60  0000 C CNN
+F 1 "SST39SF040" H 5900 7050 60  0000 C CNN
 F 2 "My_Components:IC_DIP32_600" H 6300 5800 60  0001 C CNN
 F 3 "" H 6300 5800 60  0000 C CNN
@@
 L power:GND #PWR0123
 U 1 1 5DF35AC6
-P 6300 3850
-F 0 "#PWR0123" H 6300 3600 50  0001 C CNN
-F 1 "GND" H 6300 3700 50  0000 C CNN
-F 2 "" H 6300 3850 50  0001 C CNN
-F 3 "" H 6300 3850 50  0001 C CNN
-	1    6300 3850
-	1    0    0    -1
-$EndComp
-Wire Wire Line
-	6300 3750 6300 3850
+P 6300 3800
+F 0 "#PWR0123" H 6300 3550 50  0001 C CNN
+F 1 "GND" H 6300 3650 50  0000 C CNN
+F 2 "" H 6300 3800 50  0001 C CNN
+F 3 "" H 6300 3800 50  0001 C CNN
+	1    6300 3800
+	1    0    0    -1
+$EndComp
+Wire Wire Line
+	6300 3700 6300 3800
 $Comp
 L power:GND #PWR0124
 U 1 1 5DF5154F
-P 6300 7350
-F 0 "#PWR0124" H 6300 7100 50  0001 C CNN
-F 1 "GND" H 6300 7200 50  0000 C CNN
-F 2 "" H 6300 7350 50  0001 C CNN
-F 3 "" H 6300 7350 50  0001 C CNN
-	1    6300 7350
-	1    0    0    -1
-$EndComp
-Wire Wire Line
-	6300 7250 6300 7350
-Wire Wire Line
-	6300 850  6300 750
+P 6300 7300
+F 0 "#PWR0124" H 6300 7050 50  0001 C CNN
+F 1 "GND" H 6300 7150 50  0000 C CNN
+F 2 "" H 6300 7300 50  0001 C CNN
+F 3 "" H 6300 7300 50  0001 C CNN
+	1    6300 7300
+	1    0    0    -1
+$EndComp
+Wire Wire Line
+	6300 7200 6300 7300
+Wire Wire Line
+	6300 900  6300 800
 $Comp
 L power:VCC #PWR0125
 U 1 1 5DF89883
-P 6300 750
-F 0 "#PWR0125" H 6300 600 50  0001 C CNN
-F 1 "VCC" H 6300 900 50  0000 C CNN
-F 2 "" H 6300 750 50  0001 C CNN
-F 3 "" H 6300 750 50  0001 C CNN
-	1    6300 750
-	1    0    0    -1
-$EndComp
-Wire Wire Line
-	6300 4350 6300 4250
+P 6300 800
+F 0 "#PWR0125" H 6300 650 50  0001 C CNN
+F 1 "VCC" H 6300 950 50  0000 C CNN
+F 2 "" H 6300 800 50  0001 C CNN
+F 3 "" H 6300 800 50  0001 C CNN
+	1    6300 800
+	1    0    0    -1
+$EndComp
+Wire Wire Line
+	6300 4400 6300 4300
 $Comp
 L power:VCC #PWR0126
 U 1 1 5DFA53FD
-P 6300 4250
-F 0 "#PWR0126" H 6300 4100 50  0001 C CNN
-F 1 "VCC" H 6300 4400 50  0000 C CNN
-F 2 "" H 6300 4250 50  0001 C CNN
-F 3 "" H 6300 4250 50  0001 C CNN
-	1    6300 4250
-	1    0    0    -1
-$EndComp
+P 6300 4300
+F 0 "#PWR0126" H 6300 4150 50  0001 C CNN
+F 1 "VCC" H 6300 4450 50  0000 C CNN
+F 2 "" H 6300 4300 50  0001 C CNN
+F 3 "" H 6300 4300 50  0001 C CNN
+	1    6300 4300
+	1    0    0    -1
+$EndComp
