File: Keyboard/KiCad/Omega-Keyboard.kicad_pcb (KiCad board)
At the start: 2 copper layers, 333.4 x 124.5 mm, 96 parts, among them J1 KEYBOARD, SW1 0, SW10 9, SW11 MINUS, SW12 EQUALS, SW13 BACK_SLASH, SW14 LEFT_BRACKET, SW15 RIGHT_BRACKET, SW16 SEMICOLON, SW17 QUOTE, SW18 TILDE, SW19 COMMA, SW2 1, SW20 PERIOD, SW21 SLASH, SW22 DEAD, SW23 A, SW24 B, SW25 C, SW26 D, SW27 E, SW28 F, SW29 G, SW3 2, SW30 H, SW31 I, SW32 J, SW33 K, SW34 L, SW35 M, SW36 N, SW37 O, SW38 P, SW39 Q, SW4 3, SW40 R, SW41 S, SW42 T, SW43 U, SW44 V, SW45 W, SW46 X, SW47 Y, SW48 Z, SW49 SHIFT, SW5 4, SW50 CTRL, SW51 GRAPH, SW52 CAPS_LOCK, SW53 CODE/KANA, SW54 F1/F6, SW55 F2/F7, SW56 F3/F8, SW57 F4/F9, SW58 F5/F10, SW59 ESC, SW6 5, SW60 TAB, SW61 STOP, SW62 BACK_SPACE, SW63 SELECT, SW64 RETURN, SW65 SPACE, SW66 HOME/CLS, SW67 INSERT, SW68 DELETE, SW69 LEFT, SW7 6, SW70 UP, SW71 DOWN, SW72 RIGHT, SW73 SHIFT, SW8 7, SW9 8, U1 74LS145, U2 74LS07

Commit message: Keyboard: PCB v1.1 updates
Signed-off-by: Sergey Kiselev <skiselev@gmail.com>
Parts:
- removed RR1: 4.7k, My_Components:Conn_SIL10
- added REF**: Symbol_GNU-Logo_SilkscreenTop, Symbol:Symbol_GNU-Logo_SilkscreenTop, F.Cu at (353.1, 163.8)
- added REF**: OSHW-Logo_7.5x8mm_SilkScreen, Symbol:OSHW-Logo_7.5x8mm_SilkScreen, F.Cu at (337.8, 163.8)
- added RN1: 4.7k, My_Components:Conn_SIL6, F.Cu at (228.6, 110.5)
Routing:
- net /COLUMN3: track 566.5 -> 479.1 mm
- net /COLUMN1: track 610.0 -> 622.2 mm, vias 2 -> 1
- net /COLUMN4: track 610.1 -> 606.1 mm
- net /D3+: track 140.8 -> 138.5 mm
- net /KANA_LED_BUFFERED: track 161.7 -> 159.6 mm
- net /COLUMN2: track 612.6 -> 611.6 mm
Other:
- board text added: "Omega Home Computer Keyboard - Version 1.1 Copyright (C) 2018, 2020 Sergey Kiselev"
- board text added: "github.com/skiselev/omega www.malinov.com"
- board text removed: "Omega Home Computer Keyboard - Version 1.0 Copyright (C) 2018 Sergey Kiselev"
