File: Keyboard/KiCad/Omega-Keyboard.sch (KiCad schematic (older format))
At the start: 96 parts, among them J1 KEYBOARD, SW1 0, SW10 9, SW11 MINUS, SW12 EQUALS, SW13 BACK_SLASH, SW14 LEFT_BRACKET, SW15 RIGHT_BRACKET, SW16 SEMICOLON, SW17 QUOTE, SW18 TILDE, SW19 COMMA, SW2 1, SW20 PERIOD, SW21 SLASH, SW22 DEAD, SW23 A, SW24 B, SW25 C, SW26 D, SW27 E, SW28 F, SW29 G, SW3 2, SW30 H, SW31 I, SW32 J, SW33 K, SW34 L, SW35 M, SW36 N, SW37 O, SW38 P, SW39 Q, SW4 3, SW40 R, SW41 S, SW42 T, SW43 U, SW44 V, SW45 W, SW46 X, SW47 Y, SW48 Z, SW49 SHIFT, SW5 4, SW50 CTRL, SW51 GRAPH, SW52 CAPS_LOCK, SW53 CODE/KANA, SW54 F1/F6, SW55 F2/F7, SW56 F3/F8, SW57 F4/F9, SW58 F5/F10, SW59 ESC, SW6 5, SW60 TAB, SW61 STOP, SW62 BACK_SPACE, SW63 SELECT, SW64 RETURN, SW65 SPACE, SW66 HOME/CLS, SW67 INSERT, SW68 DELETE, SW69 LEFT, SW7 6, SW70 UP, SW71 DOWN, SW72 RIGHT, SW73 SHIFT, SW8 7, SW9 8, U1 74LS145, U2 74LS07

Commit message: Keyboard: PCB v1.1 updates
Signed-off-by: Sergey Kiselev <skiselev@gmail.com>
Parts:
- removed RR1: 4.7k, My_Components:Conn_SIL10, symbol RR9
- removed U2: 74LS07, My_Components:IC_DIP14_300, symbol 74LS07
- added RN1: 4.7k, My_Components:Conn_SIL6, symbol Device:R_Network05
- added U2: 74LS07, My_Components:IC_DIP14_300, symbol Omega-Keyboard-rescue:74LS07
- C1, C2: symbol C -> Device:C
- C3: symbol CP1 -> Device:CP1
- D1, D2, D3: symbol LED-RESCUE-MSX-Keyboard -> Device:LED
- D4, D5, D6: symbol D -> Device:D
- HOLE1, HOLE2, HOLE3, HOLE4, HOLE5, HOLE6, HOLE7: symbol HOLE -> my_components:HOLE
- J1: symbol CONN_02X08 -> Connector_Generic:Conn_02x08_Odd_Even
- R1, R2, R3: symbol R -> Device:R
- SW1, SW10, SW11, SW12, SW13, SW14, SW15, SW16, SW17, SW18, SW19, SW2, SW20, SW21, SW22, SW23, SW24, SW25, SW26, SW27, SW28, SW29, SW3, SW30, SW31, SW32, SW33, SW34, SW35, SW36, SW37, SW38, SW39, SW4, SW40, SW41, SW42, SW43, SW44, SW45, SW46, SW47, SW48, SW49, SW5, SW50, SW51, SW52, SW53, SW54, SW55, SW56, SW57, SW58, SW59, SW6, SW60, SW61, SW62, SW63, SW64, SW65, SW66, SW67, SW68, SW69, SW7, SW70, SW71, SW72, SW73, SW8, SW9: symbol SW_PUSH_SMALL -> Switch:SW_Push_45deg
- U1: symbol 74LS145 -> 74xx:74LS145
Connections:
- net CAPS_LED: now also U2.13
- net CAPS_LED_BUFFERED: now also U2.12
- net COLUMN0: now also RN1.3 (R2), U2.5
- net COLUMN0_BUF: now also U2.6
- net COLUMN2: now also RN1.4 (R3), U2.3
- net COLUMN2_BUF: now also U2.4
- net COLUMN4: now also RN1.5 (R4), U2.1
- net COLUMN4_BUF: now also U2.2
- net GND: now also U2.7 (GND), U2.7 (GND), U2.7 (GND), U2.7 (GND), U2.7 (GND), U2.7 (GND)
- net KANA_LED: now also U2.11
- net KANA_LED_BUFFERED: now also U2.10
- net ROW6: now also U2.8
- net ROW6_UNBUF: now also RN1.2 (R1), U2.9
- net VCC: now also RN1.1 (common), U2.14 (VCC), U2.14 (VCC), U2.14 (VCC), U2.14 (VCC), U2.14 (VCC), U2.14 (VCC)
- no-connect marks 1 -> 2
Other:
- moved on the sheet: R1, R2, R3
